File: KiCad/weatherStation.kicad_pcb (KiCad board)
At the start: 2 copper layers, 78.8 x 64.5 mm, 7 parts, among them SW1 RotaryEncoder_Switch, U1 TFT_ST7735_SD, U2 WEMOS_C3_Mini

Commit message: Add images
Parts:
- added G***: LOGO, LOGO, F.Cu at (173.8, 76.4)
Routing:
- net Net-(U2-RX): track 71.9 -> 73.4 mm
- net Net-(U2-TX): track 82.2 -> 83.6 mm
Other:
- board text added: "3XAY"
